Commit message: Kinect properties file replaced by macro parameters

File: common_sensors/urdf/sensors/kinect.urdf.xacro (robot description, xacro)
@@ -2,10 +2,9 @@
 <root name="sensor_kinect" xmlns:xacro="http://ros.org/wiki/xacro">
 	<xacro:include filename="$(find common_sensors)/urdf/sensors/kinect_gazebo.xacro" />
-  <xacro:include filename="$(find common_sensors)/urdf/sensors/kinect_properties.urdf.xacro"/>
   <!-- camera_name has to be unique! -->
   <xacro:kinect_sensor link_name="camera_depth_frame" camera_name="camera1"
                        frame_name="camera_depth_optical_frame"/>
-	<!-- Parameterised in part by the values in kinect_properties.urdf.xacro -->
-	<xacro:macro name="sensor_kinect" params="parent">
+	<!-- Parameterised by translation and rotation of camera from its base link -->
+	<xacro:macro name="sensor_kinect" params="parent cam_px:=0 cam_py:=0 cam_pz:=0 cam_or:=0 cam_op:=0 cam_oy:=0">
 		<joint name="camera_rgb_joint" type="fixed">
 		      <origin xyz="${cam_px} ${cam_py} ${cam_pz}"
